File: Platine/Car/Car.kicad_sch (KiCad schematic)
At the start: 24 parts, among them J1 MOTOR_L, J2 Arducam_Connector1, J3 Arducam_Connector2, J4 MOTOR_R, Q1 TN0702N3, Q11 TN0702N3, Q12 TN0702N3, Q13 TN0702N3, Q14 TN0702N3, Q2 LP0701N3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

Commit message: First verion on pcb tested and functional.
Parts:
- C1, C5, C6: footprint Connector_PinHeader_2.54mm:PinHeader_1x08_P2.54mm_Vertical -> Capacitor_THT:CP_Radial_D5.0mm_P2.50mm
- C2: footprint Capacitor_THT:C_Disc_D4.3mm_W1.9mm_P5.00mm -> Capacitor_THT:CP_Radial_D5.0mm_P2.50mm
Other:
- note added: "Power Amplifier for left Motor"
- note added: "Power Amplifier for right Motor"
- note removed: "Power Amplifiers for Motors"
